Commit message: lots of changes to how stuff is organized, not yet tested
Signed-off-by: Justin Lopato <justin@lopato.org>

File: robots/servobot_description/urdf/robot.urdf (robot description, URDF)
Before this commit: robot servobot, 13 links, 12 joints
Joints:
- joint bl_bot: limit lower=-1.5708 upper=1.5708 effort=10 velocity=10 -> lower=-1.5708 upper=1.5708 effort=2 velocity=7
- joint bl_hip: limit lower=-1 upper=1 effort=10 velocity=10 -> lower=-1 upper=1 effort=2 velocity=7
- joint bl_top: limit lower=-1.5708 upper=1.5708 effort=10 velocity=10 -> lower=-1.5708 upper=1.5708 effort=2 velocity=7
- joint br_bot: limit lower=-1.5708 upper=1.5708 effort=10 velocity=10 -> lower=-1.5708 upper=1.5708 effort=2 velocity=7
- joint br_hip: limit lower=-1 upper=1 effort=10 velocity=10 -> lower=-1 upper=1 effort=2 velocity=7
- joint br_top: limit lower=-1.5708 upper=1.5708 effort=10 velocity=10 -> lower=-1.5708 upper=1.5708 effort=2 velocity=7
- joint fl_bot: limit lower=-1.5708 upper=1.5708 effort=10 velocity=10 -> lower=-1.5708 upper=1.5708 effort=2 velocity=7
- joint fl_hip: limit lower=-1 upper=1 effort=10 velocity=10 -> lower=-1 upper=1 effort=2 velocity=7
- joint fl_top: limit lower=-1.5708 upper=1.5708 effort=10 velocity=10 -> lower=-1.5708 upper=1.5708 effort=2 velocity=7
- joint fr_bot: limit lower=-1.5708 upper=1.5708 effort=10 velocity=10 -> lower=-1.5708 upper=1.5708 effort=2 velocity=7
- joint fr_hip: limit lower=-1 upper=1 effort=10 velocity=10 -> lower=-1 upper=1 effort=2 velocity=7
- joint fr_top: limit lower=-1.5708 upper=1.5708 effort=10 velocity=10 -> lower=-1.5708 upper=1.5708 effort=2 velocity=7
